Commit message: initial commit 9/3/2024

File: champ_description/urdf/spot/camera.xacro (robot description, xacro)
@@ -46,5 +46,21 @@
                         </lens>
                     </camera>
-                    <plugin filename="mono-camera-system" name="subt::MonoCameraSystem" />
+                    <plugin filename="mono-camera-system" name="subt::MonoCameraSystem" >
+                    <!--added by diya 8/30-->
+                        <camera>
+                            <image_topic>camera/image_raw</image_topic>
+                            <camera_info_topic>camera/camera_info</camera_info_topic>
+                            <frame_name>camera_frame</frame_name>
+                            <update_rate>30.0</update_rate>
+                        </camera>
+                    </plugin>
+                    <!-- <plugin name="camera_controller" filename="libgazebo_ros_camera.so">
+                        <ros>
+                            <namespace>custom_ns</namespace>
+                            <argument>image_raw:=custom</argument>
+                            <argument>camera_info:=custom_info</argument>
+                        </ros>
+                            <hack_baseline>0.07</hack_baseline>
+                    </plugin> -->
                 </sensor>
                 <sensor name="${name}_depth" type="depth_camera">

File: champ_description/urdf/spot/spot.urdf.xacro (robot description, xacro)
@@ -137,20 +137,63 @@
     <xacro:spot_camera prefix="$(arg prefix)" name="back" simulate="$(arg simulate_cameras)" />
     <xacro:fixed_joint name="camera_back_j" parent="$(arg prefix)base_link" child="$(arg prefix)camera_back" xyz="-0.425 0 0.01" rpy="0 0.3 ${-pi}" />
-    <gazebo>
-        <plugin name="p3d_base_controller" filename="libgazebo_ros_p3d.so">
-            <ros>
-                <namespace></namespace>
-                <remapping>odom:=odom/ground_truth</remapping>
-            </ros>
-            <body_name>base_link</body_name>
-            <update_rate>20</update_rate>
-            <xyz_offset>0 0 0</xyz_offset>
-            <rpy_offset>0.0 0.0 0.0</rpy_offset>
-            <gaussian_noise>0.01</gaussian_noise>
-        </plugin>
-    </gazebo>
-    <gazebo>
-        <plugin name="gazebo_ros2_control" filename="libgazebo_ros2_control.so">
+    <ros2_control name="IgnitionSystem" type="system">
+        <hardware>
+            <plugin>ign_ros2_control/IgnitionSystem</plugin>
+        </hardware>
+        <joint name="front_left_hip_x">
+            <command_interface name="position"/>
+            <state_interface name="position"/>
+        </joint>
+        <joint name="front_left_hip_y">
+            <command_interface name="position"/>
+            <state_interface name="position"/>
+        </joint>
+        <joint name="front_left_knee">
+            <command_interface name="position"/>
+            <state_interface name="position"/>
+        </joint>
+        <joint name="front_right_hip_x">
+            <command_interface name="position"/>
+            <state_interface name="position"/>
+        </joint>
+        <joint name="front_right_hip_y">
+            <command_interface name="position"/>
+            <state_interface name="position"/>
+        </joint>
+        <joint name="front_right_knee">
+            <command_interface name="position"/>
+            <state_interface name="position"/>
+        </joint>
+        <joint name="rear_left_hip_x">
+            <command_interface name="position"/>
+            <state_interface name="position"/>
+        </joint>
+        <joint name="rear_left_hip_y">
+            <command_interface name="position"/>
+            <state_interface name="position"/>
+        </joint>
+        <joint name="rear_left_knee">
+            <command_interface name="position"/>
+            <state_interface name="position"/>
+        </joint>
+        <joint name="rear_right_hip_x">
+            <command_interface name="position"/>
+            <state_interface name="position"/>
+        </joint>
+        <joint name="rear_right_hip_y">
+            <command_interface name="position"/>
+            <state_interface name="position"/>
+        </joint>
+        <joint name="rear_right_knee">
+            <command_interface name="position"/>
+            <state_interface name="position"/>
+        </joint>
+    </ros2_control>
+   <gazebo>
+        <plugin name="ign_ros2_control::IgnitionROS2ControlPlugin" filename="ign_ros2_control-system">
+            <!-- <robot_param>robot_description</robot_param> -->
+            <!-- <robot_param_node>robot_state_publisher</robot_param_node> -->
             <parameters>$(find champ_bringup)/config/ros2_control_spot.yaml</parameters>
+            <!-- <controller_manager_name>controller_manager</controller_manager_name> -->
         </plugin>
     </gazebo>

Commit message: clock synced

File: champ_description/urdf/spot/camera.xacro (robot description, xacro)
@@ -46,6 +46,6 @@
                         </lens>
                     </camera>
-                    <plugin filename="mono-camera-system" name="subt::MonoCameraSystem" >
-                    <!--added by diya 8/30-->
+                    <plugin filename="libmono_camera_system.so" name="subt::MonoCameraSystem" >
+                     <!-- added by diya 8/30  -->
                         <camera>
                             <image_topic>camera/image_raw</image_topic>
@@ -55,12 +55,4 @@
                         </camera>
                     </plugin>
-                    <!-- <plugin name="camera_controller" filename="libgazebo_ros_camera.so">
-                        <ros>
-                            <namespace>custom_ns</namespace>
-                            <argument>image_raw:=custom</argument>
-                            <argument>camera_info:=custom_info</argument>
-                        </ros>
-                            <hack_baseline>0.07</hack_baseline>
-                    </plugin> -->
                 </sensor>
                 <sensor name="${name}_depth" type="depth_camera">

File: champ_description/urdf/spot/spot.urdf.xacro (robot description, xacro)
@@ -141,59 +141,120 @@
             <plugin>ign_ros2_control/IgnitionSystem</plugin>
         </hardware>
+            <!--Front left joints-->
         <joint name="front_left_hip_x">
-            <command_interface name="position"/>
-            <state_interface name="position"/>
+            <command_interface name="position">
+               <param name="min">-${pi}</param>
+                <param name="max">${pi}</param>
+            </command_interface>
+            <state_interface name="position" />
+            <state_interface name="velocity" />
+            <state_interface name="effort" />
         </joint>
         <joint name="front_left_hip_y">
-            <command_interface name="position"/>
-            <state_interface name="position"/>
+            <command_interface name="position">
+                <param name="min">-${pi}</param>
+                <param name="max">${pi}</param>
+            </command_interface>
+            <state_interface name="position" />
+            <state_interface name="velocity" />
+            <state_interface name="effort" />
         </joint>
         <joint name="front_left_knee">
-            <command_interface name="position"/>
-            <state_interface name="position"/>
-        </joint>
+            <command_interface name="position">
+                <param name="min">-${pi}</param>
+                <param name="max">${pi}</param>
+            </command_interface>
+            <state_interface name="position" />
+            <state_interface name="velocity" />
+            <state_interface name="effort" />
+        </joint>
+        <!-- front right joints-->
         <joint name="front_right_hip_x">
-            <command_interface name="position"/>
-            <state_interface name="position"/>
+            <command_interface name="position">
+                <param name="min">-${pi}</param>
+                <param name="max">${pi}</param>
+            </command_interface>
+            <state_interface name="position" />
+            <state_interface name="velocity" />
+            <state_interface name="effort" />
         </joint>
         <joint name="front_right_hip_y">
-            <command_interface name="position"/>
-            <state_interface name="position"/>
+            <command_interface name="position">
+                <param name="min">-${pi}</param>
+                <param name="max">${pi}</param>
+            </command_interface>
+            <state_interface name="position" />
+            <state_interface name="velocity" />
+            <state_interface name="effort" />
         </joint>
         <joint name="front_right_knee">
-            <command_interface name="position"/>
-            <state_interface name="position"/>
-        </joint>
+            <command_interface name="position">
+                <param name="min">-${pi}</param>
+                <param name="max">${pi}</param>
+            </command_interface>
+            <state_interface name="position" />
+            <state_interface name="velocity" />
+            <state_interface name="effort" />
+        </joint>
+        <!--Rear Left joints-->
         <joint name="rear_left_hip_x">
-            <command_interface name="position"/>
-            <state_interface name="position"/>
+            <command_interface name="position">
+                <param name="min">-${pi}</param>
+                <param name="max">${pi}</param>
+            </command_interface>
+            <state_interface name="position" />
+            <state_interface name="velocity" />
+            <state_interface name="effort" />
         </joint>
         <joint name="rear_left_hip_y">
-            <command_interface name="position"/>
-            <state_interface name="position"/>
+            <command_interface name="position">
+                <param name="min">-${pi}</param>
+                <param name="max">${pi}</param>
+            </command_interface>
+            <state_interface name="position" />
+            <state_interface name="velocity" />
+            <state_interface name="effort" />
         </joint>
         <joint name="rear_left_knee">
-            <command_interface name="position"/>
-            <state_interface name="position"/>
-        </joint>
+            <command_interface name="position">
+                <param name="min">-${pi}</param>
+                <param name="max">${pi}</param>
+            </command_interface>
+            <state_interface name="position" />
+            <state_interface name="velocity" />
+            <state_interface name="effort" />
+        </joint>
+        <!--Rear Right joints-->
         <joint name="rear_right_hip_x">
-            <command_interface name="position"/>
-            <state_interface name="position"/>
+            <command_interface name="position">
+                <param name="min">-${pi}</param>
+                <param name="max">${pi}</param>
+            </command_interface>
+            <state_interface name="position" />
+            <state_interface name="velocity" />
+            <state_interface name="effort" />
         </joint>
         <joint name="rear_right_hip_y">
-            <command_interface name="position"/>
-            <state_interface name="position"/>
+            <command_interface name="position">
+                <param name="min">-${pi}</param>
+                <param name="max">${pi}</param>
+            </command_interface>
+            <state_interface name="position" />
+            <state_interface name="velocity" />
+            <state_interface name="effort" />
         </joint>
         <joint name="rear_right_knee">
-            <command_interface name="position"/>
-            <state_interface name="position"/>
+             <command_interface name="position">
+                <param name="min">-${pi}</param>
+                <param name="max">${pi}</param>
+            </command_interface>
+            <state_interface name="position" />
+            <state_interface name="velocity" />
+            <state_interface name="effort" />
         </joint>
     </ros2_control>
    <gazebo>
         <plugin name="ign_ros2_control::IgnitionROS2ControlPlugin" filename="ign_ros2_control-system">
-            <!-- <robot_param>robot_description</robot_param> -->
-            <!-- <robot_param_node>robot_state_publisher</robot_param_node> -->
             <parameters>$(find champ_bringup)/config/ros2_control_spot.yaml</parameters>
-            <!-- <controller_manager_name>controller_manager</controller_manager_name> -->
         </plugin>
     </gazebo>

File: champ_description/urdf/spot/spot_leg.urdf.xacro (robot description, xacro)
@@ -157,36 +157,4 @@
             </actuator>
         </transmission>
-        <ros2_control name="GazeboSystem" type="system">
-            <hardware>
-                <plugin>gazebo_ros2_control/GazeboSystem</plugin>
-            </hardware>
-            <joint name="${leg_name}_hip_x">
-                <command_interface name="position">
-                    <param name="min">-${pi}</param>
-                    <param name="max">${pi}</param>
-                </command_interface>
-                <state_interface name="position" />
-                <state_interface name="velocity" />
-                <state_interface name="effort" />
-            </joint>
-            <joint name="${leg_name}_hip_y">
-                <command_interface name="position">
-                    <param name="min">-${pi}</param>
-                    <param name="max">${pi}</param>
-                </command_interface>
-                <state_interface name="position" />
-                <state_interface name="velocity" />
-                <state_interface name="effort" />
-            </joint>
-            <joint name="${leg_name}_knee">
-                <command_interface name="position">
-                    <param name="min">-${pi}</param>
-                    <param name="max">${pi}</param>
-                </command_interface>
-                <state_interface name="position" />
-                <state_interface name="velocity" />
-                <state_interface name="effort" />
-            </joint>
-        </ros2_control>
     </xacro:macro>
 </robot>

Commit message: space ros challenge 9/10

File: champ_description/urdf/spot/camera.xacro (robot description, xacro)
@@ -47,5 +47,5 @@
                     </camera>
                     <plugin filename="libmono_camera_system.so" name="subt::MonoCameraSystem" >
-                     <!-- added by diya 8/30  -->
+                     <!-- added by diya 8/30
                         <camera>
                             <image_topic>camera/image_raw</image_topic>
@@ -53,5 +53,5 @@
                             <frame_name>camera_frame</frame_name>
                             <update_rate>30.0</update_rate>
-                        </camera>
+                        </camera>  -->
                     </plugin>
                 </sensor>

File: champ_description/urdf/spot/spot.urdf.xacro (robot description, xacro)
@@ -9,5 +9,5 @@
     </xacro:unless>
     <!-- Pass either "urdf" or "ign" to tell the parser what is the desired target format. -->
-    <xacro:arg name="rendering_target" default="urdf" />
+    <xacro:arg name="rendering_target" default="ign" />
     <xacro:arg name="simulate_cameras" default="False" />
     <xacro:arg name="simulate_imu" default="False" />
@@ -22,10 +22,10 @@
         <visual>
             <geometry>
-                <mesh filename="$(find champ_description)/meshes/spot/body.dae" />
+                <mesh filename="file://$(find champ_description)/meshes/spot/body.dae" />
             </geometry>
         </visual>
         <collision>
             <geometry>
-                <mesh filename="$(find champ_description)/meshes/spot/body_collision.stl" />
+                <mesh filename="file://$(find champ_description)/meshes/spot/body_collision.stl" />
             </geometry>
         </collision>

File: champ_description/urdf/spot/spot_leg.urdf.xacro (robot description, xacro)
@@ -130,8 +130,8 @@
             <type>transmission_interface/SimpleTransmission</type>
             <joint name="${leg_name}_hip_x">
-                <hardwareInterface>hardware_interface/EffortJointInterface</hardwareInterface>
+                <hardwareInterface>hardware_interface/VelocityJointInterface</hardwareInterface>
             </joint>
             <actuator name="${leg_name}_hip_x_actuator">
-                <hardwareInterface>hardware_interface/EffortJointInterface</hardwareInterface>
+                <hardwareInterface>hardware_interface/VelocityJointInterface</hardwareInterface>
                 <mechanicalReduction>1</mechanicalReduction>
             </actuator>
@@ -140,8 +140,8 @@
             <type>transmission_interface/SimpleTransmission</type>
             <joint name="${leg_name}_hip_y">
-                <hardwareInterface>hardware_interface/EffortJointInterface</hardwareInterface>
+                <hardwareInterface>hardware_interface/VelocityJointInterface</hardwareInterface>
             </joint>
             <actuator name="${leg_name}_hip_y_actuator">
-                <hardwareInterface>hardware_interface/EffortJointInterface</hardwareInterface>
+                <hardwareInterface>hardware_interface/VelocityJointInterface</hardwareInterface>
                 <mechanicalReduction>1</mechanicalReduction>
             </actuator>
@@ -150,8 +150,8 @@
             <type>transmission_interface/SimpleTransmission</type>
             <joint name="${leg_name}_knee">
-                <hardwareInterface>hardware_interface/EffortJointInterface</hardwareInterface>
+                <hardwareInterface>hardware_interface/VelocityJointInterface</hardwareInterface>
             </joint>
             <actuator name="${leg_name}_knee_actuator">
-                <hardwareInterface>hardware_interface/EffortJointInterface</hardwareInterface>
+                <hardwareInterface>hardware_interface/VelocityJointInterface</hardwareInterface>
                 <mechanicalReduction>1</mechanicalReduction>
             </actuator>
